Commit message: update osoyoo urdf

File: onga_description/urdf/osoyoo.urdf.xacro (robot description, xacro)
@@ -1,4 +1,4 @@
 <?xml version="1.0"?>
-<robot xmlns:xacro="http://www.ros.org/wiki/xacro" name="soma">
+<robot name="osoyoo" xmlns:xacro="http://www.ros.org/wiki/xacro" >
 	<!--  -->
 	<!--  -->
@@ -8,4 +8,26 @@
 	<!--  -->
 	<!--  -->
+	<material name="gray">
+		<color rgba="0.5 0.5 0.5 2.5"/>
+	</material>
+	<material name="red">
+		<color rgba="1.0 0.0 0.0 2.5"/>
+	</material>
+	<xacro:macro name="wheel_macro" params="parent prefix xyz">
+		<joint name="${prefix}_joint" type="continuous">
+		<origin xyz="${xyz}" rpy="${radians(-90)} 0 0"/>
+		<parent link="${parent}"/>
+		<child  link="${prefix}_link"/>
+		<axis xyz="0 0 1" />
+		</joint>
+		<link name="${prefix}_link">
+			<visual>
+				<geometry>
+					<cylinder radius="0.033" length="0.025" />
+				</geometry>
+				<material name="red"/>
+			</visual>
+		</link>
+  	</xacro:macro>
 	<link name="base_link">
 		<visual>
@@ -21,9 +43,27 @@
 		<parent link="base_link" />
 		<child link="base_footprint" />
-		<origin xyz="0.0 0.0 -0.006" rpy="0.0 0.0 0.0" />
+		<origin xyz="0.0 0.0 -0.03" rpy="0.0 0.0 0.0" />
 	</joint>
+	<joint name="body_joint" type="fixed">
+		<parent link="base_link"/>
+		<child  link="body_link"/>
+		<origin xyz="0.0 0.0 0.057" rpy="0 0 0"/>
+  	</joint>
+	<link name="body_link">
+		<visual>
+			<origin xyz="0 0 0" rpy="0 0 0" />
+			<geometry>
+				<box size="0.11 0.115 0.114" />
+			</geometry>
+			<material name="gray" />
+		</visual>
+ 	 </link>
+	<xacro:wheel_macro prefix="left_front_wheel"  parent="base_link" xyz="0.05 0.07 0.0"/>
+	<xacro:wheel_macro prefix="right_front_wheel" parent="base_link" xyz="0.05 -0.07 0.0"/>
+	<xacro:wheel_macro prefix="left_rear_wheel"  parent="base_link" xyz="-0.05 0.07 0.0"/>
+	<xacro:wheel_macro prefix="right_rear_wheel" parent="base_link" xyz="-0.05 -0.07 0.0"/>
 	<!--
 	sensor links
-	D435,VLP-16,IMU, ...
+	D435,T265 ...
 	-->
 	<!-- realsense link (front side) -->
@@ -37,13 +77,3 @@
 		<origin xyz="0.0 0.0 0.0" rpy="0.0 0.1745 0.0" />
 	</sensor_d435>
-	<!-- realsense link (rear side) -->
-	<!-- <link name="camera_r_mount_link" />
-	<joint name="camera_r_mount_joint" type="fixed">
-		<parent link="base_link" />
-		<child link="camera_r_mount_link" />
-		<origin xyz="-0.2 0.0 0.35" rpy="0.0 0.0 -3.1415" />
-	</joint>
-	<sensor_d435 parent="camera_r_mount_link" name="camera_r">
-		<origin xyz="0.0 0.0 0.0" rpy="0.0 0.2617 0.0" />
-	</sensor_d435> -->
 </robot>

Commit message: fix onga_rs

File: onga_description/urdf/osoyoo.urdf.xacro (robot description, xacro)
@@ -68,11 +68,11 @@
 	-->
 	<!-- realsense link (front side) -->
-	<link name="camera_f_mount_link" />
-	<joint name="camera_f_mount_joint" type="fixed">
+	<link name="camera_mount_link" />
+	<joint name="camera_mount_joint" type="fixed">
 		<parent link="base_link" />
-		<child link="camera_f_mount_link" />
+		<child link="camera_mount_link" />
 		<origin xyz="0.087 0.0 0.097" rpy="0.0 0.0 0.0" />
 	</joint>
-	<sensor_d435 parent="camera_f_mount_link" name="camera_f">
+	<sensor_d435 parent="camera_mount_link" name="d400">
 		<origin xyz="0.0 0.0 0.0" rpy="0.0 0.1745 0.0" />
 	</sensor_d435>

Commit message: update osoyoo urdf

File: onga_description/urdf/osoyoo.urdf.xacro (robot description, xacro)
@@ -1,11 +1,13 @@
 <?xml version="1.0"?>
 <robot name="osoyoo" xmlns:xacro="http://www.ros.org/wiki/xacro" >
-	<!--  -->
-	<!--  -->
-	<include filename="$(find realsense2_description)/urdf/_d435.urdf.xacro" />
-	<!-- <include filename="$(find velodyne_description)/urdf/VLP-16.urdf.xacro" /> -->
-	<!--  -->
-	<!--  -->
-	<!--  -->
+	<!-- load sensor models -->
+	<!-- <include filename="$(find realsense2_description)/urdf/_d435.urdf.xacro" /> -->
+	<xacro:include filename="$(find husky_description)/urdf/accessories/intel_realsense.urdf.xacro"/>
+	<!-- parameters -->
+	<xacro:arg name="rs_mount_xyz" default="0.087 0.0 0.097" />
+  	<xacro:arg name="rs_mount_rpy" default="0.0 0.0 0.0" />
+	<xacro:arg name="d435_xyz" default="0.0 0.0 0.0" />
+  	<xacro:arg name="d435_rpy" default="0.0 0.1745 0.0" />
+	<!-- define colors and materials -->
 	<material name="gray">
 		<color rgba="0.5 0.5 0.5 2.5"/>
@@ -30,13 +32,10 @@
 		</link>
   	</xacro:macro>
+	<!-- define TF links -->
 	<link name="base_link">
 		<visual>
 			<origin xyz="0.06 0.0 0.0" rpy="0.0 0.0 0.0" />
-			<!-- <geometry>
-				<box size="0.25 0.11 0.17" />
-			</geometry> -->
 		</visual>
 	</link>
-	<!-- Base footprint is on the ground under the robot -->
 	<link name="base_footprint" />
 	<joint name="base_footprint_joint" type="fixed">
@@ -63,17 +62,13 @@
 	<xacro:wheel_macro prefix="rear_left_wheel_link"  parent="base_link" xyz="-0.05 0.07 0.0"/>
 	<xacro:wheel_macro prefix="rear_right_wheel_link" parent="base_link" xyz="-0.05 -0.07 0.0"/>
-	<!--
-	sensor links
-	D435,T265 ...
-	-->
-	<!-- realsense link (front side) -->
-	<link name="camera_mount_link" />
-	<joint name="camera_mount_joint" type="fixed">
+	<link name="rs_mount_link" />
+	<joint name="rs_mount_joint" type="fixed">
 		<parent link="base_link" />
-		<child link="camera_mount_link" />
-		<origin xyz="0.087 0.0 0.097" rpy="0.0 0.0 0.0" />
+		<child link="rs_mount_link" />
+		<origin xyz="$(arg rs_mount_xyz)" rpy="$(arg rs_mount_rpy)" />
 	</joint>
-	<sensor_d435 parent="camera_mount_link" name="d400">
-		<origin xyz="0.0 0.0 0.0" rpy="0.0 0.1745 0.0" />
-	</sensor_d435>
+	<!-- <sensor_d435 parent="rs_mount_link" name="camera">
+		<origin xyz="$(arg d435_xyz)" rpy="$(arg d435_rpy)" />
+	</sensor_d435> -->
+	<xacro:intel_realsense_mount prefix="camera" topic="realsense" parent_link="rs_mount_link"/>
 </robot>

Commit message: update osoyoo urdf2

File: onga_description/urdf/osoyoo.urdf.xacro (robot description, xacro)
@@ -2,11 +2,11 @@
 <robot name="osoyoo" xmlns:xacro="http://www.ros.org/wiki/xacro" >
 	<!-- load sensor models -->
-	<!-- <include filename="$(find realsense2_description)/urdf/_d435.urdf.xacro" /> -->
-	<xacro:include filename="$(find husky_description)/urdf/accessories/intel_realsense.urdf.xacro"/>
+	<include filename="$(find realsense2_description)/urdf/_d435.urdf.xacro" />
+	<!-- <xacro:include filename="$(find husky_description)/urdf/accessories/intel_realsense.urdf.xacro"/> -->
 	<!-- parameters -->
 	<xacro:arg name="rs_mount_xyz" default="0.087 0.0 0.097" />
   	<xacro:arg name="rs_mount_rpy" default="0.0 0.0 0.0" />
-	<xacro:arg name="d435_xyz" default="0.0 0.0 0.0" />
-  	<xacro:arg name="d435_rpy" default="0.0 0.1745 0.0" />
+	<xacro:arg name="d400_xyz" default="0.0 0.0 0.0" />
+  	<xacro:arg name="d400_rpy" default="0.0 0.1745 0.0" />
 	<!-- define colors and materials -->
 	<material name="gray">
@@ -68,7 +68,7 @@
 		<origin xyz="$(arg rs_mount_xyz)" rpy="$(arg rs_mount_rpy)" />
 	</joint>
-	<!-- <sensor_d435 parent="rs_mount_link" name="camera">
-		<origin xyz="$(arg d435_xyz)" rpy="$(arg d435_rpy)" />
-	</sensor_d435> -->
-	<xacro:intel_realsense_mount prefix="camera" topic="realsense" parent_link="rs_mount_link"/>
+	<sensor_d435 parent="rs_mount_link" name="d400">
+		<origin xyz="$(arg d400_xyz)" rpy="$(arg d400_rpy)" />
+	</sensor_d435>
+	<!-- <xacro:intel_realsense_mount prefix="camera" topic="realsense" parent_link="rs_mount_link"/> -->
 </robot>

Commit message: update robot description (osoyoo)

File: onga_description/urdf/osoyoo.urdf.xacro (robot description, xacro)
@@ -3,10 +3,11 @@
 	<!-- load sensor models -->
 	<include filename="$(find realsense2_description)/urdf/_d435.urdf.xacro" />
-	<!-- <xacro:include filename="$(find husky_description)/urdf/accessories/intel_realsense.urdf.xacro"/> -->
 	<!-- parameters -->
 	<xacro:arg name="rs_mount_xyz" default="0.087 0.0 0.097" />
   	<xacro:arg name="rs_mount_rpy" default="0.0 0.0 0.0" />
-	<xacro:arg name="d400_xyz" default="0.0 0.0 0.0" />
-  	<xacro:arg name="d400_rpy" default="0.0 0.1745 0.0" />
+	<!-- <xacro:arg name="d400_xyz" default="0.0 0.0 0.0" />
+  	<xacro:arg name="d400_rpy" default="0.0 0.1745 0.0" /> -->
+	<xacro:arg name="t265_xyz" default="0.0 0.0 0.025" />
+  	<xacro:arg name="t265_rpy" default="0.0 0.0 0.0" />
 	<!-- define colors and materials -->
 	<material name="gray">
@@ -63,12 +64,27 @@
 	<xacro:wheel_macro prefix="rear_right_wheel_link" parent="base_link" xyz="-0.05 -0.07 0.0"/>
 	<link name="rs_mount_link" />
-	<joint name="rs_mount_joint" type="fixed">
+	<joint name="mount_base_joint" type="fixed">
 		<parent link="base_link" />
 		<child link="rs_mount_link" />
 		<origin xyz="$(arg rs_mount_xyz)" rpy="$(arg rs_mount_rpy)" />
 	</joint>
-	<sensor_d435 parent="rs_mount_link" name="d400">
+	<link name="t265_odom_frame"/>
+	<joint name="t265_mount_joint" type="fixed">
+		<origin xyz="$(arg t265_xyz)" rpy="$(arg t265_rpy)"/>
+		<parent link="rs_mount_link"/>
+		<child link="t265_odom_frame"/>
+	</joint>
+	<!-- <link name="t265_link"/>
+	<sensor_d435 parent="t265_link" name="d400">
+		<origin xyz="0.0 0.0 0.0" rpy="0.0 0.0 0.0" />
+	</sensor_d435> -->
+	<!-- <sensor_d435 parent="rs_mount_link" name="d400">
 		<origin xyz="$(arg d400_xyz)" rpy="$(arg d400_rpy)" />
 	</sensor_d435>
-	<!-- <xacro:intel_realsense_mount prefix="camera" topic="realsense" parent_link="rs_mount_link"/> -->
+	<link name="t265_odom_frame"/>
+	<joint name="t265_d400" type="fixed">
+		<origin xyz="0.00 0.0 0.00" rpy="0.0 -0.1745 0.0"/>
+		<parent link="d400_link"/>
+		<child link="t265_odom_frame"/>
+	</joint> -->
 </robot>

Commit message: fix tf_links

File: onga_description/urdf/osoyoo.urdf.xacro (robot description, xacro)
@@ -8,5 +8,5 @@
 	<!-- <xacro:arg name="d400_xyz" default="0.0 0.0 0.0" />
   	<xacro:arg name="d400_rpy" default="0.0 0.1745 0.0" /> -->
-	<xacro:arg name="t265_xyz" default="0.0 0.0 0.025" />
+	<xacro:arg name="t265_xyz" default="0.0 0.0 0.015" />
   	<xacro:arg name="t265_rpy" default="0.0 0.0 0.0" />
 	<!-- define colors and materials -->
@@ -75,16 +75,3 @@
 		<child link="t265_odom_frame"/>
 	</joint>
-	<!-- <link name="t265_link"/>
-	<sensor_d435 parent="t265_link" name="d400">
-		<origin xyz="0.0 0.0 0.0" rpy="0.0 0.0 0.0" />
-	</sensor_d435> -->
-	<!-- <sensor_d435 parent="rs_mount_link" name="d400">
-		<origin xyz="$(arg d400_xyz)" rpy="$(arg d400_rpy)" />
-	</sensor_d435>
-	<link name="t265_odom_frame"/>
-	<joint name="t265_d400" type="fixed">
-		<origin xyz="0.00 0.0 0.00" rpy="0.0 -0.1745 0.0"/>
-		<parent link="d400_link"/>
-		<child link="t265_odom_frame"/>
-	</joint> -->
 </robot>

Commit message: fix tf_links2

File: onga_description/urdf/osoyoo.urdf.xacro (robot description, xacro)
@@ -6,8 +6,6 @@
 	<xacro:arg name="rs_mount_xyz" default="0.087 0.0 0.097" />
   	<xacro:arg name="rs_mount_rpy" default="0.0 0.0 0.0" />
-	<!-- <xacro:arg name="d400_xyz" default="0.0 0.0 0.0" />
-  	<xacro:arg name="d400_rpy" default="0.0 0.1745 0.0" /> -->
-	<xacro:arg name="t265_xyz" default="0.0 0.0 0.015" />
-  	<xacro:arg name="t265_rpy" default="0.0 0.0 0.0" />
+	<xacro:arg name="d400_xyz" default="0.0 0.0 0.0" />
+  	<xacro:arg name="d400_rpy" default="0.0 0.1745 0.0" />
 	<!-- define colors and materials -->
 	<material name="gray">
@@ -69,9 +67,6 @@
 		<origin xyz="$(arg rs_mount_xyz)" rpy="$(arg rs_mount_rpy)" />
 	</joint>
-	<link name="t265_odom_frame"/>
-	<joint name="t265_mount_joint" type="fixed">
-		<origin xyz="$(arg t265_xyz)" rpy="$(arg t265_rpy)"/>
-		<parent link="rs_mount_link"/>
-		<child link="t265_odom_frame"/>
-	</joint>
+	<sensor_d435 parent="rs_mount_link" name="d400">
+		<origin xyz="$(arg d400_xyz)" rpy="$(arg d400_rpy)" />
+	</sensor_d435>
 </robot>

Commit message: update params for costmap

File: onga_description/urdf/osoyoo.urdf.xacro (robot description, xacro)
@@ -4,5 +4,5 @@
 	<include filename="$(find realsense2_description)/urdf/_d435.urdf.xacro" />
 	<!-- parameters -->
-	<xacro:arg name="rs_mount_xyz" default="0.087 0.0 0.097" />
+	<xacro:arg name="rs_mount_xyz" default="0.087 0.0 0.08" />
   	<xacro:arg name="rs_mount_rpy" default="0.0 0.0 0.0" />
 	<xacro:arg name="d400_xyz" default="0.0 0.0 0.0" />
@@ -34,5 +34,5 @@
 	<link name="base_link">
 		<visual>
-			<origin xyz="0.06 0.0 0.0" rpy="0.0 0.0 0.0" />
+			<origin xyz="0.0 0.0 0.0" rpy="0.0 0.0 0.0" />
 		</visual>
 	</link>

Commit message: fix urdf

File: onga_description/urdf/osoyoo.urdf.xacro (robot description, xacro)
@@ -32,9 +32,5 @@
   	</xacro:macro>
 	<!-- define TF links -->
-	<link name="base_link">
-		<visual>
-			<origin xyz="0.0 0.0 0.0" rpy="0.0 0.0 0.0" />
-		</visual>
-	</link>
+	<link name="base_link"/>
 	<link name="base_footprint" />
 	<joint name="base_footprint_joint" type="fixed">
